File: throwing-star.sch (KiCad schematic (older format))
At the start: 6 parts, among them J1 RJ45, J2 RJ45, J3 RJ45, J4 RJ45

Commit message: update project using kicad (5.1.6)-1
Parts:
- C1, C2: footprint (none) -> Capacitor_THT:C_Disc_D3.0mm_W1.6mm_P2.50mm; symbol C -> Device:C_Small
- J1, J2, J3, J4: footprint (none) -> Connector_RJ:RJ45_Amphenol_RJHSE5380; symbol RJ45 -> Connector:8P8C_Shielded
Connections:
- wire segments 40 -> 64
